File: stm32-debug-breakout.kicad_pcb (KiCad board)
At the start: 2 copper layers, 21.6 x 48.3 mm, 5 parts, among them J1 FTDI, J2 STLINK, J3 ST_PROGRAM_DEBUG, SW1 SW_MEC_5E

Commit message: 2021-10-24
Connections:
- J1 pad 4: /RX -> /TX
- J1 pad 5: /TX -> /RX
Routing:
- net /RX: track 34.0 -> 40.4 mm
- net /TX: track 31.8 -> 30.8 mm

Commit message: 2021-10-24
Other:
- net class Default: clearance 0.2 -> 0.1778; trace_width 0.25 -> 0.2286; via_dia 0.8 -> 0.7874; via_drill 0.4 -> 0.381
- rule pad_to_mask_clearance: 0 -> 0.0508
- rule trace_clearance: 0.2 -> 0.1778
- rule trace_min: 0.2 -> 0.1778
- rule via_min_drill: 0.3 -> 0.3048
- rule via_min_size: 0.4 -> 0.5588
